File: hardware/Dot.sch (EAGLE design)
At the start: 25 parts, among them IC1 CAT24M010TS, U1 ATMEGA328P-MU-QFN32, U2 TMP102

Commit message: v0.5
Parts:
- removed SJ3: (no value), SparkFun:SOLDERJUMPER_2WAYS
- removed U$3: MPU-9250, invensense:MPU-9250
- added C4, C8: 0.1uF, resistor:C-EUC0603
- added C5, C7: (no value), resistor:C-EUC0603
- added C6: 1uF, resistor:C-EUC0603
- added IC2: SI1145, silabs:SI1145
- added L1: 3.3µH/±20%/450mA, SparkFun-Coils:INDUCTOR-0805-3.3UH
- added SJ5: (no value), SparkFun:SOLDERJUMPER_2WAYS
- added U3: ISL29125, SparkFun-Sensors:ISL29125
- added U4: 9DoF IMU, SparkFun-Sensors:MPU-9250
- R3: value 1kΩ -> 10kΩ
Connections:
- removed net ANT_2: ANT1.1, SJ2.2
- removed net N$8: C2.1, U$3.REGOUT
- new net ANT: ANT1.1, C5.1, L1.1, SJ2.2
- new net INT_RGB: U1.PB6(XTAL1/TOSC1/PCINT6), U3.!INT
- new net INT_UV: IC2.INT, U1.PB7(XTAL2/TOSC2/PCINT7)
- new net N$11: C8.1, U4.REGOUT
- new net N$14: SJ5.2, U4.AD0/SDO
- net +3V3: now also C2.1, C4.1, C6.1, IC2.VDD, JP2.3, SJ5.3, U3.VDD, U4.VDD; no longer JP2.2, SJ3.3, U$3.VDD
- net GND: now also C4.2, C5.2, C6.2, C7.2, C8.2, IC2.GND, JP2.4, SJ5.1, U3.GND, U4.GND; no longer JP2.1, SJ3.1, U$3.GND
- net MOVE_INT: now also U4.INT; no longer U$3.INT
- net N$9: now also C7.1, L1.2; no longer SJ3.2, U$3.ADO/SDO
- net SCL: now also IC2.SCL, JP2.2, U3.SCL, U4.SCL/SCLK; no longer JP2.4, U$3.SCL/SCLK
- net SDA: now also IC2.SDA, JP2.1, U3.SDA, U4.SDA/SDI; no longer JP2.3, U$3.SDA/SDI
Other:
- note added: "E2PROM"
- note added: "Light RGB"
- note added: "Light UV"
- note added: "Light intensity"
- note added: "MCU"
- note added: "Movement"
- note added: "Radio"
- note added: "Temperature / Humidity"
- note removed: "Leave pad unsoldered for increased accuracy"
- moved on the sheet: ANT1, BAT1, C1, C2, C3, IC1, JP2, JP3, LED1, R1, R2, R3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

Commit message: udpating schematic
Other:
- note added: "Analog Light"
- note added: "Antenna Tuning"
- note added: "Headers"
- note added: "I2C, Reset and Push Pullups"
- moved on the sheet: C1, C5, C6, C7, L1, U3
Changed lines of the file:
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@@
 <wire x1="223.52" y1="-2.54" x2="223.52" y2="-83.82" width="0.1524" layer="95" style="longdash"/>
 <wire x1="312.42" y1="-2.54" x2="312.42" y2="-83.82" width="0.1524" layer="95" style="longdash"/>
-<text x="71.12" y="-10.16" size="3.81" layer="95">Movement</text>
-<text x="152.4" y="-83.82" size="3.81" layer="95">Temperature / Humidity</text>
-<text x="259.08" y="-83.82" size="3.81" layer="95">Light UV</text>
-<wire x1="-50.8" y1="5.08" x2="317.5" y2="5.08" width="0.1524" layer="95" style="longdash"/>
+<text x="58.42" y="-81.28" size="3.81" layer="95">Movement</text>
+<text x="152.4" y="-81.28" size="3.81" layer="95">Temperature / Humidity</text>
+<text x="261.62" y="-81.28" size="3.81" layer="95">Light UV</text>
+<wire x1="-50.8" y1="5.08" x2="388.62" y2="5.08" width="0.1524" layer="95" style="longdash"/>
 <wire x1="10.16" y1="-2.54" x2="10.16" y2="-83.82" width="0.1524" layer="95" style="longdash"/>
 <text x="-43.18" y="-81.28" size="3.81" layer="95">Light intensity</text>
 <wire x1="223.52" y1="93.98" x2="223.52" y2="12.7" width="0.1524" layer="95" style="longdash"/>
 <wire x1="129.54" y1="93.98" x2="129.54" y2="12.7" width="0.1524" layer="95" style="longdash"/>
-<wire x1="17.78" y1="101.6" x2="317.5" y2="101.6" width="0.1524" layer="95" style="longdash"/>
+<wire x1="-48.26" y1="101.6" x2="388.62" y2="101.6" width="0.1524" layer="95" style="longdash"/>
 <wire x1="223.52" y1="190.5" x2="223.52" y2="109.22" width="0.1524" layer="95" style="longdash"/>
 <wire x1="129.54" y1="190.5" x2="129.54" y2="109.22" width="0.1524" layer="95" style="longdash"/>
 <wire x1="10.16" y1="93.98" x2="10.16" y2="12.7" width="0.1524" layer="95" style="longdash"/>
-<text x="66.04" y="12.7" size="3.81" layer="95">E2PROM</text>
+<text x="66.04" y="10.16" size="3.81" layer="95">E2PROM</text>
 <text x="172.72" y="10.16" size="3.81" layer="95">MCU</text>
-<text x="259.08" y="12.7" size="3.81" layer="95">Radio</text>
-<text x="370.84" y="-76.2" size="3.81" layer="95">Light RGB</text>
+<text x="259.08" y="10.16" size="3.81" layer="95">Radio</text>
+<text x="347.98" y="-81.28" size="3.81" layer="95">Light RGB</text>
 <wire x1="312.42" y1="93.98" x2="312.42" y2="12.7" width="0.1524" layer="95" style="longdash"/>
+<text x="-38.1" y="10.16" size="3.81" layer="95">Analog Light</text>
+<text x="340.36" y="10.16" size="3.81" layer="95">Antenna Tuning</text>
+<text x="60.96" y="106.68" size="3.81" layer="95">Headers</text>
+<text x="238.76" y="106.68" size="3.81" layer="95">I2C, Reset and Push Pullups</text>
 </plain>
 <instances>
@@
 <instance part="IC2" gate="G$1" x="274.32" y="-25.4"/>
 <instance part="SUPPLY20" gate="GND" x="264.16" y="-38.1" rot="MR0"/>
-<instance part="U3" gate="G$1" x="381" y="-17.78"/>
-<instance part="C6" gate="G$1" x="360.68" y="-17.78"/>
-<instance part="SUPPLY21" gate="GND" x="360.68" y="-25.4" rot="MR0"/>
+<instance part="U3" gate="G$1" x="358.14" y="-27.94"/>
+<instance part="C6" gate="G$1" x="337.82" y="-27.94"/>
+<instance part="SUPPLY21" gate="GND" x="337.82" y="-35.56" rot="MR0"/>
 <instance part="U4" gate="G$1" x="78.74" y="-27.94"/>
 <instance part="SUPPLY23" gate="GND" x="60.96" y="-35.56"/>
@@
 <instance part="C8" gate="G$1" x="50.8" y="-33.02"/>
 <instance part="SUPPLY25" gate="GND" x="50.8" y="-40.64"/>
-<instance part="+3V9" gate="G$1" x="350.52" y="-12.7"/>
-<instance part="C1" gate="G$1" x="350.52" y="-17.78"/>
-<instance part="SUPPLY10" gate="GND" x="350.52" y="-25.4"/>
+<instance part="+3V9" gate="G$1" x="327.66" y="-22.86"/>
+<instance part="C1" gate="G$1" x="327.66" y="-27.94"/>
+<instance part="SUPPLY10" gate="GND" x="327.66" y="-35.56"/>
 <instance part="+3V10" gate="G$1" x="243.84" y="-12.7"/>
 <instance part="C2" gate="G$1" x="243.84" y="-17.78"/>
@@
 <instance part="C4" gate="G$1" x="33.02" y="-22.86"/>
 <instance part="SUPPLY13" gate="GND" x="33.02" y="-30.48"/>
-<instance part="C5" gate="G$1" x="350.52" y="78.74"/>
-<instance part="C7" gate="G$1" x="365.76" y="78.74"/>
-<instance part="SUPPLY16" gate="GND" x="360.68" y="68.58"/>
-<instance part="L1" gate="G$1" x="358.14" y="81.28" rot="R90"/>
+<instance part="C5" gate="G$1" x="350.52" y="53.34"/>
+<instance part="C7" gate="G$1" x="365.76" y="53.34"/>
+<instance part="SUPPLY16" gate="GND" x="360.68" y="43.18"/>
+<instance part="L1" gate="G$1" x="358.14" y="55.88" rot="R90"/>
 </instances>
 <busses>
@@
 <pinref part="C6" gate="G$1" pin="2"/>
 <pinref part="U3" gate="G$1" pin="GND"/>
-<wire x1="360.68" y1="-22.86" x2="370.84" y2="-22.86" width="0.1524" layer="91"/>
-<wire x1="370.84" y1="-22.86" x2="370.84" y2="-20.32" width="0.1524" layer="91"/>
-<junction x="360.68" y="-22.86"/>
+<wire x1="337.82" y1="-33.02" x2="347.98" y2="-33.02" width="0.1524" layer="91"/>
+<wire x1="347.98" y1="-33.02" x2="347.98" y2="-30.48" width="0.1524" layer="91"/>
+<junction x="337.82" y="-33.02"/>
 <pinref part="SUPPLY21" gate="GND" pin="GND"/>
 </segment>
@@
 <pinref part="C5" gate="G$1" pin="2"/>
 <pinref part="SUPPLY16" gate="GND" pin="GND"/>
-<wire x1="350.52" y1="73.66" x2="350.52" y2="71.12" width="0.1524" layer="91"/>
-<wire x1="350.52" y1="71.12" x2="360.68" y2="71.12" width="0.1524" layer="91"/>
-<wire x1="360.68" y1="71.12" x2="365.76" y2="71.12" width="0.1524" layer="91"/>
-<junction x="360.68" y="71.12"/>
+<wire x1="350.52" y1="48.26" x2="350.52" y2="45.72" width="0.1524" layer="91"/>
+<wire x1="350.52" y1="45.72" x2="360.68" y2="45.72" width="0.1524" layer="91"/>
+<wire x1="360.68" y1="45.72" x2="365.76" y2="45.72" width="0.1524" layer="91"/>
+<junction x="360.68" y="45.72"/>
 <pinref part="C7" gate="G$1" pin="2"/>
-<wire x1="365.76" y1="71.12" x2="365.76" y2="73.66" width="0.1524" layer="91"/>
+<wire x1="365.76" y1="45.72" x2="365.76" y2="48.26" width="0.1524" layer="91"/>
 </segment>
 </net>
@@
 <segment>
 <pinref part="U3" gate="G$1" pin="SDA"/>
-<wire x1="391.16" y1="-15.24" x2="393.7" y2="-15.24" width="0.1524" layer="91"/>
-<label x="393.7" y="-15.24" size="1.27" layer="95" xref="yes"/>
+<wire x1="368.3" y1="-25.4" x2="370.84" y2="-25.4" width="0.1524" layer="91"/>
+<label x="370.84" y="-25.4" size="1.27" layer="95" xref="yes"/>
 </segment>
 <segment>
@@
 <pinref part="C6" gate="G$1" pin="1"/>
 <pinref part="U3" gate="G$1" pin="VDD"/>
-<wire x1="360.68" y1="-15.24" x2="370.84" y2="-15.24" width="0.1524" layer="91"/>
-<wire x1="350.52" y1="-15.24" x2="360.68" y2="-15.24" width="0.1524" layer="91"/>
-<junction x="350.52" y="-15.24"/>
-<junction x="360.68" y="-15.24"/>
+<wire x1="337.82" y1="-25.4" x2="347.98" y2="-25.4" width="0.1524" layer="91"/>
+<wire x1="327.66" y1="-25.4" x2="337.82" y2="-25.4" width="0.1524" layer="91"/>
+<junction x="327.66" y="-25.4"/>
+<junction x="337.82" y="-25.4"/>
 </segment>
 <segment>
@@
 <segment>
 <pinref part="U3" gate="G$1" pin="SCL"/>
-<wire x1="391.16" y1="-17.78" x2="393.7" y2="-17.78" width="0.1524" layer="91"/>
-<label x="393.7" y="-17.78" size="1.27" layer="95" xref="yes"/>
+<wire x1="368.3" y1="-27.94" x2="370.84" y2="-27.94" width="0.1524" layer="91"/>
+<label x="370.84" y="-27.94" size="1.27" layer="95" xref="yes"/>
 </segment>
 <segment>
@@
 <segment>
 <pinref part="C5" gate="G$1" pin="1"/>
-<wire x1="350.52" y1="81.28" x2="342.9" y2="81.28" width="0.1524" layer="91"/>
-<label x="342.9" y="81.28" size="1.27" layer="95" rot="R180" xref="yes"/>
+<wire x1="350.52" y1="55.88" x2="342.9" y2="55.88" width="0.1524" layer="91"/>
+<label x="342.9" y="55.88" size="1.27" layer="95" rot="R180" xref="yes"/>
 <pinref part="L1" gate="G$1" pin="1"/>
-<wire x1="353.06" y1="81.28" x2="350.52" y2="81.28" width="0.1524" layer="91"/>
-<junction x="350.52" y="81.28"/>
+<wire x1="353.06" y1="55.88" x2="350.52" y2="55.88" width="0.1524" layer="91"/>
+<junction x="350.52" y="55.88"/>
 </segment>
 </net>
@@
 <segment>
 <pinref part="U3" gate="G$1" pin="!INT"/>
-<wire x1="391.16" y1="-20.32" x2="393.7" y2="-20.32" width="0.1524" layer="91"/>
-<label x="393.7" y="-20.32" size="1.27" layer="95" xref="yes"/>
+<wire x1="368.3" y1="-30.48" x2="370.84" y2="-30.48" width="0.1524" layer="91"/>
+<label x="370.84" y="-30.48" size="1.27" layer="95" xref="yes"/>
 </segment>
 <segment>
@@
 <pinref part="C7" gate="G$1" pin="1"/>
 <pinref part="L1" gate="G$1" pin="2"/>
-<wire x1="363.22" y1="81.28" x2="365.76" y2="81.28" width="0.1524" layer="91"/>
-</segment>
-</net>
+<wire x1="363.22" y1="55.88" x2="365.76" y2="55.88" width="0.1524" layer="91"/>
+</segment>
+</net>

Commit message: v1.3
Parts:
- removed JP3: (no value), pinhead:PINHD-1X8
- removed R1: 150Ω, resistor:R-EU_R0603
- added JP1: (no value), pinhead:PINHD-1X10
- added R5: 130Ω, resistor:R-EU_R0603
- added R6, R8: 30Ω, resistor:R-EU_R0603
- added SPK1: SMT-0540-S-R, adafruit:SMT-0540-S-R
- added U$3: AT45DB641E, AT45DB641E:AT45DB641E
- added U$4: LDCL015, LDCL015:LDCL015
- added U5: BMP18, Seeed-OPL-sensor:PRESSURE-BMP180(LGA7)
- LED1: value (none) -> GM1WA55311A; device SparkFun:LED0603 -> led:GM1WA55311A
Connections:
- removed net ADC1: JP3.2, R4.1, U1.PC1(ADC1PCINT9)
- removed net N$7: LED1.A, R1.2
- new net ADC: JP1.2, R4.1, U1.ADC6
- new net BUZZER: SPK1.-, U1.PC0(ADC0/PCINT8)
- new net FLASH_CS: U$3.CS, U1.PC1(ADC1PCINT9)
- new net N$1: LED1.CBLUE, R8.1
- new net N$15: LED1.CGREEN, R5.1
- new net RXD: JP1.4, R5.2, U1.PD0(RXD/PCINT16)
- new net VIN: JP1.6, U$4.ENA, U$4.VIN
- net +3V3: now also LED1.A, U$3.NRST, U$3.VCC, U$4.OUT, U1.AVCC, U4.VDDIO, U5.VDD, U5.VDDIO; no longer JP3.4
- net GND: now also JP1.5, SPK1.+, SW1.2, U$3.GND, U$3.PAD, U$4.GND, U4.FSYNC, U5.GND; no longer JP3.3, LED1.C, R7A.2
- net LED: now also R8.2; no longer R1.1
- net LIGHT_SENSE: now also U1.ADC7; no longer U1.PC0(ADC0/PCINT8)
- net MISO: now also JP1.9, U$3.SO; no longer JP3.7
- net MOSI: now also JP1.10, U$3.SI; no longer JP3.8
- net MOVE_INT: now also U1.PC2(ADC2PCINT10); no longer U1.PD0(RXD/PCINT16)
- net N$4: now also LED1.CRED, R6.1; no longer R7A.1, SW1.2
- net PUSH: now also JP1.1, U1.PD3(INT1/OC2B/PCINT19); no longer U1.PD2(INT0/PCINT18)
- net RIRQ: now also U1.PD2(INT0/PCINT18); no longer U1.PC3(ADC3/PCINT11)
- net RSEL: now also U1.PC3(ADC3/PCINT11); no longer U1.PD3(INT1/OC2B/PCINT19)
- net RST: now also JP1.7; no longer JP3.5
- net SCK: now also JP1.8, U$3.SCK; no longer JP3.6
- net SCL: now also U5.SCL
- net SDA: now also U5.SDA
- net TXD: now also JP1.3, R6.2; no longer JP3.1
Other:
- note added: "0110000D"
- note added: "0x0A / yes"
- note added: "0x44 / yes"
- note added: "0x48 / yes, temperature-dependent values, incorrect (70 degC)"
- note added: "0x60 / yes"
- note added: "0x77 / no ??"
- note added: "1000100D"
- note added: "100100XD"
- note added: "1010XXXD"
- note added: "110100XD"
- note added: "1110111D"
- note added: "9DoF"
- note added: "Actors RGB Led, Buzzer"
- note added: "BMP18"
- note added: "Barometric pressure Temperature Humidity"
- note added: "CAT24M01"
- note added: "D = Direction"
- note added: "EEPROM 1Mbit"
- note added: "Flash & E2PROM"
- note added: "Hex Address / Tested?"
- note added: "I2C Address"
- note added: "I2C, Reset and Pullups & Push Button(s)"
- note added: "ISL29125"
- note added: "MPU9250"
- note added: "Part #"
- note added: "Power and Headers"
- note added: "RGB"
- note added: "SI1145"
- note added: "Sensor / Memory"
- note added: "TMP102 or TMP112 (high acc +/-0.5°)"
- note added: "TMP102/112"
- note added: "Temp/Pressure"
- note added: "Temperature"
- note added: "Temperature / Humidity Barometric pressure"
- note added: "Temperature Humidity"
- note added: "UV"
- note added: "Values @ 20mA."
- note added: "use AT45DB641E-MHN-Y for starndard page size (1056b/page) or AT45DB641E-MHN2B-T for binary page size (1024b/page)"
- note removed: "Analog Light"
- note removed: "E2PROM"
- note removed: "Headers"
- note removed: "I2C, Reset and Push Pullups"
- note removed: "Temperature / Humidity"

Commit message: * Corrected RGB Led layout * Added 100uF Cap. Should soften discharges up to 30mA for 1ms. * Cap recharges in 175ms.
Parts:
- removed ANT1: AN9520, Seeed-OPL-Antenna:SMD-BUILT-IN-ANTENNA-2.4GHZ(2P-9.5X2.1MM)
- removed C5, C7: (no value), resistor:C-EUC0603
- removed L1: 3.3µH/±20%/450mA, SparkFun-Coils:INDUCTOR-0805-3.3UH
- added C9: 100uf, Seeed-OPL-Capacitor:TANTALUM-SMD-100UF-6.3V(AVX-A)
Connections:
- removed net ANT: ANT1.1, C5.1, L1.1, SJ2.2
- removed net ANT_1: SJ2.1, U$1.ANT, X1.SIGNAL
- removed net N$9: C7.1, L1.2
- new net N$3: SJ2.1, U$1.ANT
- new net N$7: SJ2.2, X1.SIGNAL
- net +3V3: now also C9.+
- net GND: now also C9.-; no longer C5.2, C7.2
Other:
- note added: "0x50 & 0x51 (a16 bit) / yes"
- note added: "0x68 / yes"
- note added: "1100000D"
- note added: "Added 100uF Cap. Should soften discharge of batetry to peaks up to 30mA for 1ms. Reacharges in 175ms."
- note added: "Blue"
- note added: "Corrected RGB Led layout."
- note added: "Diff to v1.3"
- note added: "Green"
- note added: "Red"
- note removed: "0110000D"
- note removed: "0x0A / yes"
Changed lines of the file:
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@@
 <parts>
 <part name="U1" library="Seeed-OPL-ic" deviceset="MCU-ATMEGA328P-MU(QFN32)" device="" value="ATMEGA328P-MU-QFN32"/>
-<part name="ANT1" library="Seeed-OPL-Antenna" deviceset="SMD-BUILT-IN-ANTENNA-2.4GHZ(2P-9.5X2.1MM)" device="" value="AN9520"/>
 <part name="SUPPLY2" library="supply2" deviceset="GND" device=""/>
 <part name="SUPPLY3" library="supply2" deviceset="GND" device=""/>
@@
 <part name="X1" library="adafruit" deviceset="ANTENNA_U.FL" device=""/>
 <part name="SUPPLY5" library="supply2" deviceset="GND" device=""/>
-<part name="SJ2" library="SparkFun" deviceset="SOLDERJUMPER" device="TRACE"/>
 <part name="R4" library="resistor" deviceset="R-EU_" device="R0603"/>
 <part name="BAT1" library="Battery" deviceset="BATTERY" device="20PTH"/>
@@
 <part name="C4" library="resistor" deviceset="C-EU" device="C0603" value="0.1uF"/>
 <part name="SUPPLY13" library="supply2" deviceset="GND" device=""/>
-<part name="C5" library="resistor" deviceset="C-EU" device="C0603"/>
-<part name="C7" library="resistor" deviceset="C-EU" device="C0603"/>
-<part name="SUPPLY16" library="supply2" deviceset="GND" device=""/>
-<part name="L1" library="SparkFun-Coils" deviceset="INDUCTOR" device="-0805-3.3UH" value="3.3µH/±20%/450mA"/>
 <part name="SUPPLY19" library="supply2" deviceset="GND" device=""/>
 <part name="JP1" library="pinhead" deviceset="PINHD-1X10" device=""/>
@@
 <part name="LED1" library="led" deviceset="GM1WA55311A" device=""/>
 <part name="SUPPLY28" library="supply2" deviceset="GND" device=""/>
+<part name="C9" library="Seeed-OPL-Capacitor" deviceset="TANTALUM-SMD-100UF-6.3V(AVX-A)" device="" value="100uf"/>
+<part name="+3V20" library="supply1" deviceset="+3V3" device=""/>
+<part name="SUPPLY29" library="supply2" deviceset="GND" device=""/>
+<part name="SJ2" library="SparkFun" deviceset="SOLDERJUMPER" device="TRACE"/>
 </parts>
 <sheets>
@@
 <text x="43.18" y="88.9" size="1.778" layer="91">use AT45DB641E-MHN-Y for starndard page size (1056b/page)
 or AT45DB641E-MHN2B-T for binary page size (1024b/page)</text>
+<text x="-24.13" y="50.8" size="1.27" layer="91">Blue</text>
+<text x="-7.62" y="50.8" size="1.27" layer="91" rot="R90">Green</text>
+<text x="1.778" y="50.8" size="1.27" layer="91">Red</text>
 </plain>
 <instances>
 <instance part="U1" gate="G$1" x="170.18" y="60.96"/>
-<instance part="ANT1" gate="G$1" x="292.1" y="91.44" rot="R90"/>
 <instance part="SUPPLY2" gate="GND" x="27.94" y="157.48"/>
 <instance part="SUPPLY3" gate="GND" x="144.78" y="38.1" rot="R270"/>
@@
 <instance part="X1" gate="G$1" x="297.18" y="68.58" rot="R180"/>
 <instance part="SUPPLY5" gate="GND" x="302.26" y="71.12"/>
-<instance part="SJ2" gate="1" x="292.1" y="76.2" rot="R90"/>
 <instance part="R4" gate="G$1" x="66.04" y="157.48" rot="R90"/>
 <instance part="BAT1" gate="G$1" x="27.94" y="165.1" rot="R270"/>
@@
 <instance part="C4" gate="G$1" x="33.02" y="-22.86"/>
 <instance part="SUPPLY13" gate="GND" x="33.02" y="-30.48"/>
-<instance part="C5" gate="G$1" x="350.52" y="53.34"/>
-<instance part="C7" gate="G$1" x="365.76" y="53.34"/>
-<instance part="SUPPLY16" gate="GND" x="360.68" y="43.18"/>
-<instance part="L1" gate="G$1" x="358.14" y="55.88" rot="R90"/>
 <instance part="SUPPLY19" gate="GND" x="297.18" y="124.46"/>
 <instance part="JP1" gate="A" x="76.2" y="134.62"/>
@@
 <instance part="LED1" gate="G$1" x="-10.16" y="73.66"/>
 <instance part="SUPPLY28" gate="GND" x="45.72" y="-35.56"/>
+<instance part="C9" gate="G$1" x="10.16" y="162.56" rot="R270"/>
+<instance part="+3V20" gate="G$1" x="10.16" y="172.72"/>
+<instance part="SUPPLY29" gate="GND" x="10.16" y="156.21"/>
+<instance part="SJ2" gate="1" x="284.48" y="68.58"/>
 </instances>
 <busses>
@@
 </segment>
 <segment>
-<pinref part="C5" gate="G$1" pin="2"/>
-<pinref part="SUPPLY16" gate="GND" pin="GND"/>
-<wire x1="350.52" y1="48.26" x2="350.52" y2="45.72" width="0.1524" layer="91"/>
-<wire x1="350.52" y1="45.72" x2="360.68" y2="45.72" width="0.1524" layer="91"/>
-<wire x1="360.68" y1="45.72" x2="365.76" y2="45.72" width="0.1524" layer="91"/>
-<junction x="360.68" y="45.72"/>
-<pinref part="C7" gate="G$1" pin="2"/>
-<wire x1="365.76" y1="45.72" x2="365.76" y2="48.26" width="0.1524" layer="91"/>
-</segment>
-<segment>
 <pinref part="SW1" gate="G$1" pin="2"/>
 <pinref part="SUPPLY19" gate="GND" pin="GND"/>
@@
 <wire x1="45.72" y1="-27.94" x2="45.72" y2="-33.02" width="0.1524" layer="91"/>
 <pinref part="SUPPLY28" gate="GND" pin="GND"/>
+</segment>
+<segment>
+<pinref part="C9" gate="G$1" pin="-"/>
+<pinref part="SUPPLY29" gate="GND" pin="GND"/>
 </segment>
 </net>
@@
 <wire x1="-10.16" y1="76.2" x2="-10.16" y2="78.74" width="0.1524" layer="91"/>
 </segment>
+<segment>
+<pinref part="+3V20" gate="G$1" pin="+3V3"/>
+<pinref part="C9" gate="G$1" pin="+"/>
+<wire x1="10.16" y1="170.18" x2="10.16" y2="166.37" width="0.1524" layer="91"/>
+</segment>
 </net>
 <net name="ADCENA" class="0">
@@
 </segment>
 </net>
-<net name="ANT" class="0">
-<segment>
-<pinref part="SJ2" gate="1" pin="2"/>
-<pinref part="ANT1" gate="G$1" pin="1"/>
-<wire x1="292.1" y1="83.82" x2="292.1" y2="81.28" width="0.1524" layer="91"/>
-</segment>
-<segment>
-<pinref part="C5" gate="G$1" pin="1"/>
-<wire x1="350.52" y1="55.88" x2="342.9" y2="55.88" width="0.1524" layer="91"/>
-<label x="342.9" y="55.88" size="1.27" layer="95" rot="R180" xref="yes"/>
-<pinref part="L1" gate="G$1" pin="1"/>
-<wire x1="353.06" y1="55.88" x2="350.52" y2="55.88" width="0.1524" layer="91"/>
-<junction x="350.52" y="55.88"/>
-</segment>
-</net>
-<net name="ANT_1" class="0">
-<segment>
-<pinref part="SJ2" gate="1" pin="1"/>
-<pinref part="X1" gate="G$1" pin="SIGNAL"/>
-<wire x1="292.1" y1="71.12" x2="292.1" y2="68.58" width="0.1524" layer="91"/>
-<pinref part="U$1" gate="G$1" pin="ANT"/>
-<wire x1="292.1" y1="68.58" x2="276.86" y2="68.58" width="0.1524" layer="91"/>
-<junction x="292.1" y="68.58"/>
-</segment>
-</net>
 <net name="PUSH" class="0">
 <segment>
@@
 <pinref part="C8" gate="G$1" pin="1"/>
 <wire x1="60.96" y1="-30.48" x2="50.8" y2="-30.48" width="0.1524" layer="91"/>
-</segment>
-</net>
-<net name="N$9" class="0">
-<segment>
-<pinref part="C7" gate="G$1" pin="1"/>
-<pinref part="L1" gate="G$1" pin="2"/>
-<wire x1="363.22" y1="55.88" x2="365.76" y2="55.88" width="0.1524" layer="91"/>
 </segment>
 </net>
@@
 <pinref part="R6" gate="G$1" pin="1"/>
 <wire x1="-20.32" y1="68.58" x2="-20.32" y2="66.04" width="0.1524" layer="91"/>
+</segment>
+</net>
+<net name="N$3" class="0">
+<segment>
+<pinref part="U$1" gate="G$1" pin="ANT"/>
+<pinref part="SJ2" gate="1" pin="1"/>
+<wire x1="276.86" y1="68.58" x2="279.4" y2="68.58" width="0.1524" layer="91"/>
+</segment>
+</net>
+<net name="N$7" class="0">
+<segment>
+<pinref part="SJ2" gate="1" pin="2"/>
+<pinref part="X1" gate="G$1" pin="SIGNAL"/>
+<wire x1="289.56" y1="68.58" x2="292.1" y2="68.58" width="0.1524" layer="91"/>
 </segment>
 </net>
@@
 <text x="5.08" y="68.58" size="1.27" layer="91">UV</text>
 <text x="27.94" y="68.58" size="1.27" layer="91">SI1145</text>
-<text x="48.26" y="68.58" size="1.27" layer="91">0110000D</text>
+<text x="48.26" y="68.58" size="1.27" layer="91">1100000D</text>
 <text x="5.08" y="63.5" size="1.27" layer="91">Temperature</text>
 <text x="27.94" y="63.5" size="1.27" layer="91">TMP102/112</text>
@@
 <text x="27.94" y="48.26" size="1.27" layer="91">CAT24M01 </text>
 <text x="48.26" y="48.26" size="1.27" layer="91">1010XXXD</text>
-<text x="76.2" y="48.26" size="1.27" layer="91">0x0A / yes</text>
+<text x="76.2" y="48.26" size="1.27" layer="91">0x50 &amp; 0x51 (a16 bit) / yes</text>
 <text x="48.26" y="78.74" size="1.016" layer="91">D = Direction</text>
+<text x="76.2" y="58.42" size="1.27" layer="91">0x68 / yes</text>
 </plain>
 <instances>
+</instances>
+<busses>
+</busses>
+<nets>
+</nets>
+</sheet>
+<sheet>
+<plain>
+<text x="-13.97" y="88.9" size="2.54" layer="91">Diff to v1.3</text>
+<text x="-13.462" y="80.01" size="2.1844" layer="91">Corrected RGB Led layout.</text>
+<text x="-12.7" y="73.66" size="2.1844" layer="91">Added 100uF Cap. Should soften discharge of batetry to peaks up to 30mA for 1ms. Reacharges in 175ms.</text>
+</plain>
+<instances>
